Commit message: Adding collision boundary and additional parameters

File: nuturtle_description/urdf/turtlebot3_burger.urdf.xacro (robot description, xacro)
@@ -10,4 +10,5 @@
   <xacro:property name="r" value="${params['wheel_radius']}"/>
   <xacro:property name="w" value="${params['track_width']}"/>
+  <xacro:property name="cr" value="${params['collision_radius']}"/>
   <link name="${color}_base_footprint"/>
   <joint name="${color}_base_joint" type="fixed">
@@ -27,5 +28,10 @@
       <origin xyz="-0.032 0 0.070" rpy="0 0 0"/>
       <geometry>
-        <box size="0.140 0.140 0.143"/>
+        <xacro:if value="${cr==0}">
+          <box size="0.140 0.140 0.143"/>
+        </xacro:if>
+        <xacro:if value="${cr!=0}">
+          <cylinder radius="${cr}" length=".25"/>
+        </xacro:if>
       </geometry>
     </collision>

Commit message: Almost correct LiDAR simulation

File: nuturtle_description/urdf/turtlebot3_burger.urdf.xacro (robot description, xacro)
@@ -26,5 +26,5 @@
     </visual>
     <collision>
-      <origin xyz="-0.032 0 0.070" rpy="0 0 0"/>
+      <origin xyz="0 0 0.070" rpy="0 0 0"/>
       <geometry>
         <xacro:if value="${cr==0}">
